File: electronics/_autosave-otherworlds-v2.kicad_sch (KiCad schematic)
At the start: 30 parts, among them J1 Conn_01x07, J10 LED4, J11 LED5, J12 LED6, J13 LED7, J14 LED8, J15 GND, J16 5V, J17 GND, J18 24V, J19 Conn_01x02, J2 Conn_01x07, J20 LED4, J3 SN74AHCT125N, J4 SN74AHCT125N, J7 LED1, J8 LED2, J9 LED3

Commit message: fix pcb
Connections:
- net D1: now also J4.9 (3A)
- net D2: now also J4.5 (2A)
- net D3: now also J4.2 (1A)
- net D5: no longer J4.2 (1A)
- net D6: no longer J4.5 (2A)
- net D7: no longer J4.9 (3A)
Changed lines of the file:
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@@
 		)
 	)
-	(label "D7"
+	(label "D1"
 		(at 142.24 118.745 0)
 		(effects
@@
 		)
 	)
-	(label "D5"
+	(label "D3"
 		(at 119.38 108.585 180)
 		(effects
@@
 		)
 	)
-	(label "D6"
+	(label "D2"
 		(at 119.38 116.205 180)
 		(effects
