File: electronics/otherworlds-v2.kicad_pcb (KiCad board)
At the start: 2 copper layers, 98.7 x 90.9 mm, 30 parts, among them J1 Conn_01x07, J10 LED4, J11 LED5, J12 LED6, J13 LED7, J14 LED8, J15 GND, J16 5V, J17 GND, J18 24V, J19 Conn_01x02, J2 Conn_01x07, J20 LED4, J3 SN74AHCT125N, J4 SN74AHCT125N, J7 LED1, J8 LED2, J9 LED3

Commit message: fix pcb
Parts:
- R1, R2, R3, R4, R5, R6, R7, R8: footprint Resistor_THT:R_Axial_DIN0204_L3.6mm_D1.6mm_P5.08mm_Horizontal -> Resistor_THT:R_Axial_DIN0207_L6.3mm_D2.5mm_P7.62mm_Horizontal
- moved J20 31.0 mm to (92.4, 104.2), turned to 0 degrees
- moved J7 30.5 mm to (167.9, 86.4)
- moved R1 30.5 mm to (165.1, 91.4)
- moved J2 23.1 mm to (121.3, 116.4), turned to 180 degrees
- moved J1 23.1 mm to (106.1, 116.4), turned to 180 degrees
- moved R3 20.6 mm to (164.8, 60.7)
- moved J13 20.6 mm to (167.6, 96.3)
- moved J12 20.3 mm to (167.6, 127.0)
- moved J11 20.3 mm to (167.6, 116.8)
- moved J14 20.3 mm to (167.6, 106.7)
- moved R5 20.1 mm to (165.1, 121.7)
- moved R7 20.1 mm to (164.8, 101.3)
- moved R6 20.1 mm to (164.8, 131.8)
- moved J9 20.1 mm to (167.6, 56.1)
- moved R8 20.1 mm to (165.1, 111.8)
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Connections:
- J3 pad 12: /D4 -> /D7
- J3 pad 2: /D1 -> /D8
- J3 pad 5: /D2 -> /D6
- J3 pad 9: /D3 -> /D5
- J4 pad 12: /D8 -> /D4
- J4 pad 2: /D5 -> /D3
- J4 pad 5: /D6 -> /D2
- J4 pad 9: /D7 -> /D1
Routing:
- net GND: track 0.00 -> 348.9 mm
- net Net-(J3-4Y): track 29.3 -> 55.8 mm
- net /D8: track 57.4 -> 31.1 mm
- net /D1: track 14.3 -> 35.7 mm
- net /D10: track 31.9 -> 13.9 mm
- net /D6: track 25.4 -> 11.0 mm
- net /D3: track 27.6 -> 13.8 mm
- net Net-(J3-1Y): track 60.0 -> 46.9 mm, vias 0 -> 1
- net /D9: track 27.1 -> 13.9 mm
- net Net-(J3-2Y): track 50.5 -> 63.0 mm, vias 0 -> 1
- net Net-(J4-2Y): track 41.7 -> 30.7 mm
- net /D0: track 36.6 -> 47.5 mm
- net /D7: track 50.9 -> 41.3 mm
- net /D4: track 33.8 -> 24.3 mm
- net Net-(J4-4Y): track 21.7 -> 31.0 mm
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Other:
- outline, holes or cut-outs redrawn
